File: MMBCloneProMax/MMBCloneProMax.kicad_pcb (KiCad board)
At the start: 2 copper layers, 246.2 x 30 mm, 99 parts, among them J1 UJ32-C-H-G-SMT-TR, J10 Current Sense, J11 Bat1, J12 Current Sense, J13 Bat1, J14 Current Sense, J15 Bat1, J16 Current Sense, J17 Bat1, J18 Current Sense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

Commit message: drc done
Routing:
- net GND: track 2.38 -> 24.5 mm, vias 120 -> 133
- net Net-(J18-Pin_1): track 4.00 -> 6.62 mm
