File: MMBCloneProMax/MMBCloneProMax.kicad_sch (KiCad schematic)
At the start: 8 parts, among them J1 UJ32-C-H-G-SMT-TR, J2 1337009, J3 1377295

Commit message: intermediate
Parts:
- R5: value 100k -> 10k
Changed lines of the file:
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@@
 			)
 		)
-		(property "Value" "100k"
+		(property "Value" "10k"
 			(at 125.73 20.3199 0)
 			(effects
